File: Rev0/Rev0.kicad_pcb (KiCad board)
At the start: 2 copper layers, 116 x 55.2 mm, 172 parts, among them J1 TERMBLOCK_1X2, J10 Conn_01x03, J11 Conn_01x03, J12 Conn_01x03, J2 QWIIC_RIGHT_ANGLE, J4 QWIIC_RIGHT_ANGLE, J5 Conn_01x03, J6 Conn_01x03, J7 Conn_01x03, J8 Conn_01x03, J9 Conn_01x03, K1 HK4100F-DC5, K2 HK4100F-DC5, K3 HK4100F-DC5, K4 HK4100F-DC5, K5 HK4100F-DC5, K6 HK4100F-DC5, K7 HK4100F-DC5, K8 HK4100F-DC5, Q1 AOD417, Q2 MMBT2222, Q3 MMBT2222, Q4 MMBT2222, Q5 MMBT2222, Q6 MMBT2222, Q7 MMBT2222, Q8 MMBT2222, Q9 MMBT2222, U1 BME688, U10 LTV-817S, U11 LTV-817S, U12 LTV-817S, U2 TCA9406DC, U3 K7805-2000R3L, U4 TCA9554, U5 LTV-817S, U6 LTV-817S, U7 LTV-817S, U8 LTV-817S, U9 LTV-817S

Commit message: .
Parts:
- removed FRAME1: FRAME-LETTER, Qwiic_BME688:CREATIVE_COMMONS
- removed J10, J11, J12, J6, J7, J8, J9: Conn_01x03, Connector_PinHeader_2.54mm:PinHeader_1x03_P2.54mm_Vertical
- removed LOGO2: QWIIC_LOGO_5MM, Qwiic_BME688:QWIIC_5MM
- removed LOGO5 (x2): OSHW-LOGOS, Qwiic_BME688:OSHW-LOGO-S
- removed U$1, U$33: , Qwiic_BME688:#GND#0
- removed U$10, U$7: , Qwiic_BME688:GAS_SENSOR_#_BME6880
- removed U$11: , Qwiic_BME688:#ADR#0
- removed U$12: , Qwiic_BME688:DEFAULT_ADR#_0X760
- removed U$13: , Qwiic_BME688:0X770
- removed U$14, U$15: , Qwiic_BME688:#3V3#0
- removed U$16, U$2: , Qwiic_BME688:#SDO#0
- removed U$19: , Qwiic_BME688:#SDI#0
- removed U$20: , Qwiic_BME688:#SCK#0
- removed U$21, U$22: , Qwiic_BME688:##CSB##0
- removed U$3: , Qwiic_BME688:#CSB#0
- removed U$35: , Qwiic_BME688:#SDA#0
- removed U$36: , Qwiic_BME688:#SCL#0
- removed U$5: , Qwiic_BME688:PWR0
- removed U$6: , Qwiic_BME688:#I2C#0
- removed U$8: , Qwiic_BME688:#LED#0
- removed U$9: , Qwiic_BME688:0X760
- added C6: 0.1uF, Capacitor_SMD:C_0603_1608Metric, F.Cu at (65.5, 43.1)
- added C7: 47pF-5%-X7R, Capacitor_SMD:C_0603_1608Metric, F.Cu at (69.2, 48.4)
- added C8: 22uF, Capacitor_SMD:C_0603_1608Metric, F.Cu at (73.7, 48.4)
- added C9: 22uF, Capacitor_SMD:C_0603_1608Metric, F.Cu at (75.2, 48.4)
- added G***: LOGO, Graphics:qr-AirQualityControl, F.Cu at (157.7, 65.0)
- added G***: LOGO, Graphics:Hasatio_logo_micro, F.Cu at (125.7, 40.6)
- added G***: LOGO, Graphics:Hasatio_logo_mini, B.Cu at (112.5, 45.6)
- added G***: LOGO, Graphics:qr-AirQualityControl, B.Cu at (157.7, 65.0)
- added J3: Conn_01x05, Connector_PinHeader_2.54mm:PinHeader_1x05_P2.54mm_Vertical, F.Cu at (52.8, 49.5)
- added L1: 6.8uH, Inductor_SMD:L_Bourns_SRN8040TA, F.Cu at (71.5, 42.7)
- added R7: 10k, Resistor_SMD:R_0603_1608Metric, F.Cu at (64.7, 48.4)
- added R8: 158k, Resistor_SMD:R_0603_1608Metric, F.Cu at (70.7, 48.4)
- added R9: 30k, Resistor_SMD:R_0603_1608Metric, F.Cu at (72.2, 48.4)
- added Sign-RecyclBin: , OLIMEX_LOGOs-FP:LOGO_RECYCLEBIN_1, B.Cu at (160.3, 49.8)
- added Sign_Pb-Free: , OLIMEX_LOGOs-FP:LOGO_PBFREE, B.Cu at (141.7, 46.6)
- added Sign_RoHS: Val**, OLIMEX_LOGOs-FP:LOGO_ROHS_1, B.Cu at (152.1, 56.7)
- C4: value 10uF/100v -> 4.7uF-50V; footprint Capacitor_SMD:C_0805_2012Metric -> Capacitor_SMD:C_0603_1608Metric
- C5: value 10uF -> 4.7uF-50V
- J5: value Conn_01x03 -> Conn_01x05; footprint Connector_PinHeader_2.54mm:PinHeader_1x03_P2.54mm_Vertical -> Connector_PinHeader_2.54mm:PinHeader_1x05_P2.54mm_Vertical
- K1, K2, K3, K4, K5, K6, K7, K8: value HK4100F-DC5 -> G5Q-1; footprint Relay_THT:Relay_SPDT_HJR-4102 -> Relay_THT:Relay_SPDT_Omron-G5Q-1
- R14, R15, R16, R17, R18, R19, R20, R21: value 380R -> 360R
- R23, R25, R27, R29, R31, R33, R35, R37: value 10 -> 10R
- U3: value K7805-2000R3L -> AP63357; footprint Converter_DCDC:Converter_DCDC_RECOM_R-78HB-0.5L_THT -> Qwiic_BME688:V-DFN3020-13
- U4: value TCA9554 -> TCA9534A
- moved J5 156.7 mm to (153.1, 49.5), turned to 180 degrees
- moved C4 86.0 mm to (67.7, 48.4)
- moved R6 83.8 mm to (108.0, 42.5), turned to 0 degrees
- moved U3 82.9 mm to (65.0, 45.4), turned to 0 degrees
- moved K1 82.8 mm to (53.4, 63.8), turned to -90 degrees
- moved K2 82.8 mm to (66.5, 63.8), turned to -90 degrees
- moved K3 82.8 mm to (79.5, 63.8), turned to -90 degrees
- moved K4 82.8 mm to (92.6, 63.8), turned to -90 degrees
- moved K5 82.8 mm to (105.7, 63.8), turned to -90 degrees
- moved K6 82.8 mm to (118.7, 63.8), turned to -90 degrees
- moved K7 82.8 mm to (131.8, 63.8), turned to -90 degrees
- moved K8 82.8 mm to (144.8, 63.8), turned to -90 degrees
- moved J1 82.4 mm to (138.4, 46.1)
- moved C12 82.3 mm to (87.4, 43.1)
- moved R54 82.3 mm to (88.9, 43.1)
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- renumbered JP3 to ?, JP4 to ?, JP8 to ?, JP7 to ?, C6 to C10, C7 to C11, C8 to C12, D3 to D1, D1 to D10, D2 to D11, D4 to D2, D5 to D3, D6 to D4, D7 to D5, D8 to D6, D9 to D7, D10 to D8, D11 to D9, JP9 to JP1, JP10 to JP2, JP11 to JP3, JP12 to JP4, JP13 to JP5, JP14 to JP6, JP15 to JP7, JP16 to JP8, R7 to R10, R8 to R11, R9 to R12, R10 to R13, R6 to R54, R12 to R55, R13 to R56, R11 to R6
Connections:
- C5 pad 1: +5V -> VCC
- D2 pad 1: Net-(D4-K) -> Net-(D2-K)
- D2 pad 2: Net-(D4-A) -> Net-(D2-A)
- D3 pad 1: Net-(D5-K) -> Net-(D3-K)
- D3 pad 2: Net-(D5-A) -> Net-(D3-A)
- D4 pad 1: Net-(D6-K) -> Net-(D4-K)
- D4 pad 2: Net-(D6-A) -> Net-(D4-A)
- D5 pad 1: Net-(D7-K) -> Net-(D5-K)
- D5 pad 2: Net-(D7-A) -> Net-(D5-A)
- D6 pad 1: Net-(D8-K) -> Net-(D6-K)
- D6 pad 2: Net-(D8-A) -> Net-(D6-A)
- D7 pad 1: Net-(D9-K) -> Net-(D7-K)
- D7 pad 2: Net-(D9-A) -> Net-(D7-A)
- D8 pad 1: Net-(D10-K) (its old number) -> Net-(D8-K)
- D8 pad 2: Net-(D10-A) (its old number) -> Net-(D8-A)
- D9 pad 1: Net-(D11-K) (its old number) -> Net-(D9-K)
- D9 pad 2: Net-(D11-A) (its old number) -> Net-(D9-A)
- J5 pad 1: /NO0 -> +5V
- J5 pad 2: /COM0 -> /SCL_A
- J5 pad 3: /NC0 -> /SDA_A
- K1 pad 1: (no net) -> Net-(D2-K)
- K1 pad 5: Net-(D4-K) -> Net-(D2-A)
- K2 pad 1: (no net) -> Net-(D3-K)
- K2 pad 5: Net-(D5-K) -> Net-(D3-A)
- K3 pad 1: (no net) -> Net-(D4-K)
- K3 pad 5: Net-(D6-K) -> Net-(D4-A)
- K4 pad 1: (no net) -> Net-(D5-K)
- K4 pad 5: Net-(D7-K) -> Net-(D5-A)
- K5 pad 1: (no net) -> Net-(D6-K)
- K5 pad 5: Net-(D8-K) -> Net-(D6-A)
- K6 pad 1: (no net) -> Net-(D7-K)
- K6 pad 5: Net-(D9-K) -> Net-(D7-A)
- K7 pad 1: (no net) -> Net-(D8-K)
- K7 pad 5: Net-(D10-K) (its old number) -> Net-(D8-A)
- K8 pad 1: (no net) -> Net-(D9-K)
- K8 pad 5: Net-(D11-K) (its old number) -> Net-(D9-A)
- Q2 pad 3: Net-(D4-A) -> Net-(D2-A)
- Q3 pad 3: Net-(D5-A) -> Net-(D3-A)
- Q4 pad 3: Net-(D6-A) -> Net-(D4-A)
- Q5 pad 3: Net-(D7-A) -> Net-(D5-A)
- Q6 pad 3: Net-(D8-A) -> Net-(D6-A)
- Q7 pad 3: Net-(D9-A) -> Net-(D7-A)
- Q8 pad 3: Net-(D10-A) (its old number) -> Net-(D8-A)
- Q9 pad 3: Net-(D11-A) (its old number) -> Net-(D9-A)
- R23 pad 2: Net-(D4-K) -> Net-(D2-K)
- R25 pad 2: Net-(D5-K) -> Net-(D3-K)
- R27 pad 2: Net-(D6-K) -> Net-(D4-K)
- R29 pad 2: Net-(D7-K) -> Net-(D5-K)
- R31 pad 2: Net-(D8-K) -> Net-(D6-K)
- R33 pad 2: Net-(D9-K) -> Net-(D7-K)
- R35 pad 2: Net-(D10-K) (its old number) -> Net-(D8-K)
- R37 pad 2: Net-(D11-K) (its old number) -> Net-(D9-K)
- R46 pad 1: Net-(D4-A) -> Net-(D2-A)
- R47 pad 1: Net-(D5-A) -> Net-(D3-A)
- R48 pad 1: Net-(D6-A) -> Net-(D4-A)
- R49 pad 1: Net-(D7-A) -> Net-(D5-A)
- R50 pad 1: Net-(D8-A) -> Net-(D6-A)
- R51 pad 1: Net-(D9-A) -> Net-(D7-A)
- R52 pad 1: Net-(D10-A) (its old number) -> Net-(D8-A)
- R53 pad 1: Net-(D11-A) (its old number) -> Net-(D9-A)
Routing:
- net +5V: track 287.9 -> 381.3 mm, vias 14 -> 15
- net VCC: track 67.5 -> 96.9 mm, vias 0 -> 5
- net Net-(D10-K) (its old number): track 28.7 -> 0.00 mm
- net Net-(D11-K) (its old number): track 28.6 -> 0.00 mm
- net Net-(D11-A) (its old number): track 23.0 -> 0.00 mm
- net Net-(D10-A) (its old number): track 23.0 -> 0.00 mm
- net Net-(C6-Pad2): track 0.00 -> 19.4 mm
- net Net-(D3-K): track 0.00 -> 15.4 mm
- net Net-(D2-K): track 0.00 -> 15.4 mm
- net /COM4: track 27.6 -> 12.7 mm
- net Net-(D9-A): track 23.0 -> 9.27 mm
- net Net-(D5-A): track 23.0 -> 9.30 mm
- net Net-(D8-A): track 23.0 -> 9.29 mm
- net Net-(D6-A): track 23.0 -> 9.29 mm
- net Net-(D7-A): track 23.0 -> 9.29 mm
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Other:
- board size 116 x 55.2 mm -> 116 x 58.1 mm
- board text added: "+3V"
- board text added: "+5V"
- board text added: "Air Quality Control"
- board text added: "COM0"
- board text added: "COM1"
- board text added: "COM2"
- board text added: "COM3"
- board text added: "COM4"
- board text added: "COM5"
- board text added: "COM6"
- board text added: "COM7"
- board text added: "NC0"
- board text added: "NC1"
- board text added: "NC2"
- board text added: "NC3"
- board text added: "NC4"
- board text added: "NC5"
- board text added: "NC6"
- board text added: "NC7"
- board text added: "NO0"
- board text added: "NO1"
- board text added: "NO2"
- board text added: "NO3"
- board text added: "NO4"
- board text added: "NO5"
- board text added: "NO6"
- board text added: "NO7"
- board text added: "Rev.0"
- board text added: "SCL"
- board text added: "SDA"
