File: Rev0/Rev0.kicad_sch (KiCad schematic)
At the start: 148 parts, among them J1 TERMBLOCK_1X2, J10 Conn_01x03, J11 Conn_01x03, J12 Conn_01x03, J2 QWIIC_RIGHT_ANGLE, J3 CONN_06NO_SILK_NO_POP, J4 QWIIC_RIGHT_ANGLE, J5 Conn_01x03, J6 Conn_01x03, J7 Conn_01x03, J8 Conn_01x03, J9 Conn_01x03, K1 HK4100F-DC5, K2 HK4100F-DC5, K3 HK4100F-DC5, K4 HK4100F-DC5, K5 HK4100F-DC5, K6 HK4100F-DC5, K7 HK4100F-DC5, K8 HK4100F-DC5, Q1 AOD417, Q2 MMBT2222, Q3 MMBT2222, Q4 MMBT2222, Q5 MMBT2222, Q6 MMBT2222, Q7 MMBT2222, Q8 MMBT2222, Q9 MMBT2222, U1 BME688, U10 LTV-817S, U11 LTV-817S, U12 LTV-817S, U2 TCA9406DC, U3 K7805-2000R3L, U3 TCA9554, U5 LTV-817S, U6 LTV-817S, U7 LTV-817S, U8 LTV-817S, U9 LTV-817S

Commit message: .
Parts:
- removed J10, J11, J12, J5, J6, J7, J8, J9: Conn_01x03, Connector_PinHeader_2.54mm:PinHeader_1x03_P2.54mm_Vertical, symbol Connector_Generic:Conn_01x03
- removed J3: CONN_06NO_SILK_NO_POP, Qwiic_BME688:1X06_NO_SILK, symbol Qwiic_BME688-eagle-import:CONN_06NO_SILK_NO_POP
- removed JP1, JP2, JP5, JP6: FIDUCIALUFIDUCIAL, Qwiic_BME688:FIDUCIAL-MICRO, symbol Qwiic_BME688-eagle-import:FIDUCIALUFIDUCIAL
- removed JP10, JP11, JP12, JP13, JP14, JP15, JP16, JP9: HEADER-1X3_508TERM, Connector_Phoenix_MC:PhoenixContact_MC_1,5_3-G-3.5_1x03_P3.50mm_Horizontal, symbol Adafruit PowerRelay Wing-eagle-import:HEADER-1X3_508TERM
- removed K1, K2, K3, K4, K5, K6, K7, K8: HK4100F-DC5, Relay_THT:Relay_SPDT_HJR-4102, symbol Relay:TIANBO-HJR-4102-L
- removed LOGO5: OSHW-LOGOS, Qwiic_BME688:OSHW-LOGO-S, symbol Qwiic_BME688-eagle-import:OSHW-LOGOS
- removed U3: TCA9554, Package_SO:TSSOP-16_4.4x5mm_P0.65mm, symbol SparkFun_Qwiic_GPIO-eagle-import:TCA9534U
- removed U3: K7805-2000R3L, Converter_DCDC:Converter_DCDC_RECOM_R-78HB-0.5L_THT, symbol Regulator_Switching:R-78B5.0-2.0
- added C6: 0.1uF, Capacitor_SMD:C_0603_1608Metric, symbol Adafruit PCA9685 rev C-eagle-import:CAP_CERAMIC0805-NOOUTLINE
- added C7: 47pF/5%, Capacitor_SMD:C_0603_1608Metric, symbol Adafruit PCA9685 rev C-eagle-import:CAP_CERAMIC0805-NOOUTLINE
- added C8, C9: 22uF, Capacitor_SMD:C_0603_1608Metric, symbol Adafruit PCA9685 rev C-eagle-import:CAP_CERAMIC0805-NOOUTLINE
- added J3, J5: Conn_01x05, Connector_PinHeader_2.54mm:PinHeader_1x05_P2.54mm_Vertical, symbol Connector_Generic:Conn_01x05
- added JP1, JP2, JP3, JP4, JP5, JP6, JP7, JP8: HEADER-1X3_508TERM, Connector_Phoenix_MC:PhoenixContact_MC_1,5_3-G-3.5_1x03_P3.50mm_Horizontal, symbol Adafruit PowerRelay Wing-eagle-import:HEADER-1X3_508TERM
- added K1, K2, K3, K4, K5, K6, K7, K8: G5Q-1 DC5, Relay_THT:Relay_SPDT_Omron-G5Q-1, symbol Relay:G5Q-1
- added L1: 6.8uH, Inductor_SMD:L_Bourns_SRN8040TA, symbol ESP32-GATEWAY_Rev_G:L
- added R7: 10k, Resistor_SMD:R_0603_1608Metric, symbol Adafruit PCA9685 rev C-eagle-import:RESISTOR0805_NOOUTLINE
- added R8: 158k, Resistor_SMD:R_0603_1608Metric, symbol Adafruit PCA9685 rev C-eagle-import:RESISTOR0805_NOOUTLINE
- added R9: 30k, Resistor_SMD:R_0603_1608Metric, symbol Adafruit PCA9685 rev C-eagle-import:RESISTOR0805_NOOUTLINE
- added U3: AP63357, Qwiic_BME688:V-DFN3020-13, symbol SparkFun_Buck_Regulator_AP63357DV-7_BabyBuck5V-eagle-import:AP63357
- added U4: TCA9534A, Package_SO:TSSOP-16_4.4x5mm_P0.65mm, symbol Interface_Expansion:TCA9534
- C4: value 10uF/100v -> 4.7uF/35V; footprint Capacitor_SMD:C_0805_2012Metric -> Capacitor_SMD:C_0603_1608Metric
- C5: value 10uF -> 4.7uF/35V
- JP5, LED1, LED2, LED3, LED4, LED5, LED6, LED7, LED8, LED9: now left out of the parts list
- Q1: Field4 (none) -> https://jlcpcb.com/partdetail/Jsmsemi-AOD417/C6396163
- Q2, Q3, Q4, Q5, Q6, Q7, Q8, Q9: Field4 (none) -> https://jlcpcb.com/partdetail/Yongyutai-MMBT2222/C2891810
- R14, R15, R16, R17, R18, R19, R20, R21: value 380R -> 360R
- R23, R25, R27, R29, R31, R33, R35, R37: value 10 -> 10R
- U1: Field4 (none) -> https://jlcpcb.com/partdetail/BoschSensortec-BME688/C3664478
- U10, U11, U12, U5, U6, U7, U8, U9: Field4 (none) -> https://jlcpcb.com/partdetail/liteon-LTV_817S_TA1D/C114603
- U2: Field4 (none) -> https://jlcpcb.com/partdetail/TexasInstruments-TCA9406DCUR/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
- renumbered C6 to C10, C7 to C11, C8 to C12, D3 to D1, D1 to D10, D2 to D11, D4 to D2, D5 to D3, D6 to D4, D7 to D5, D8 to D6, D9 to D7, D10 to D8, D11 to D9, R7 to R10, R8 to R11, R9 to R12, R10 to R13, R6 to R54, R12 to R55, R13 to R56, R11 to R6
Connections:
- net +3.3V: now also J3.4 (Pin_4), J5.4 (Pin_4)
- net +5V: now also C7.1, C8.1, C9.1, J3.1 (Pin_1), J5.1 (Pin_1), L1.2, R8.2, U4.16 (VDD); no longer C5.1
- net A0: now also U4.1 (A0)
- net A1: now also U4.2 (A1)
- net A2: now also U4.3 (A2)
- net COM0: now also JP1.2, K1.2
- net COM1: now also JP2.2, K2.2
- net COM2: now also JP3.2, K3.2
- net COM3: now also JP4.2, K4.2
- net COM4: now also JP5.2, K5.2
- net COM5: now also JP6.2, K6.2
- net COM6: now also JP7.2, K7.2
- net COM7: now also JP8.2, K8.2
- net GND: now also C8.2, C9.2, J3.5 (Pin_5), J5.5 (Pin_5), R9.1, U3.P$4 (COMP), U3.P$8 (GND), U4.8 (GND)
- net NC0: now also JP1.3, K1.4
- net NC1: now also JP2.3, K2.4
- net NC2: now also JP3.3, K3.4
- net NC3: now also JP4.3, K4.4
- net NC4: now also JP5.3, K5.4
- net NC5: now also JP6.3, K6.4
- net NC6: now also JP7.3, K7.4
- net NC7: now also JP8.3, K8.4
- net NO0: now also JP1.1, K1.3
- net NO1: now also JP2.1, K2.3
- net NO2: now also JP3.1, K3.3
- net NO3: now also JP4.1, K4.3
- net NO4: now also JP5.1, K5.3
- net NO5: now also JP6.1, K6.3
- net NO6: now also JP7.1, K7.3
- net NO7: now also JP8.1, K8.3
- net Out0: now also U4.4 (P0)
- net Out1: now also U4.5 (P1)
- net Out2: now also U4.6 (P2)
- net Out3: now also U4.7 (P3)
- net Out4: now also U4.9 (P4)
- net Out5: now also U4.10 (P5)
- net Out6: now also U4.11 (P6)
- net Out7: now also U4.12 (P7)
- net SCL_A: now also J3.2 (Pin_2), J5.2 (Pin_2)
- net SCL_B: now also U4.14 (SCL)
- net SDA_A: now also J3.3 (Pin_3), J5.3 (Pin_3)
- net SDA_B: now also U4.15 (SDA)
- net VCC: now also C5.1, R7.2, U3.P$1 (VIN)
- net at D4.2 (A), Q4.3 (C), R48.1: now also K3.5
- net at R2.1: now also U4.13 (~{INT})
- net at D8.1 (K), R35.2: now also K7.1
- net at D8.2 (A), Q8.3 (C), R52.1: now also K7.5
- net at D5.2 (A), Q5.3 (C), R49.1: now also K4.5
- net at D7.2 (A), Q7.3 (C), R51.1: now also K6.5
- net at D5.1 (K), R29.2: now also K4.1
- net at D6.1 (K), R31.2: now also K5.1
- net at D6.2 (A), Q6.3 (C), R50.1: now also K5.5
- net at D9.2 (A), Q9.3 (C), R53.1: now also K8.5
- net at D9.1 (K), R37.2: now also K8.1
- net at D2.1 (K), R23.2: now also K1.1
- net at D3.1 (K), R25.2: now also K2.1
- net at D3.2 (A), Q3.3 (C), R47.1: now also K2.5
- net at D7.1 (K), R33.2: now also K6.1
- net at D2.2 (A), Q2.3 (C), R46.1: now also K1.5
- net at D4.1 (K), R27.2: now also K3.1
- new net: C6.2, L1.1, U3.P$7 (SW), U3.P$9 (SW)
- new net: C7.2, R8.1, R9.2, U3.P$3 (FB)
- new net: R7.1, U3.P$2 (EN)
- new net: C6.1, U3.P$6 (BST)
Other:
- note added: "Reverse voltage protection"
- note removed: "Reverse voltage"
- note removed: "protection"
- moved on the sheet: C10, C11, C12, C3, D1, D10, D11, D13, D14, D15, D17, D18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
